File: PTH PCB/HydroHAT.kicad_pcb (KiCad board)
At the start: 2 copper layers, 65 x 56 mm, 1 part

Commit message: PTH PCB Complete
Schematic also somewhat reworked.
Parts:
- removed U***: DIP-40_600, DIP-40__600
- added C1: 0.1uF, C1, F.Cu at (132.7, 120.7)
- added C2: 0.1uF, C1, F.Cu at (127.0, 79.8)
- added C3: 0.1uF, C1, F.Cu at (167.4, 110.7)
- added C4: 0.1uF, C1, F.Cu at (152.1, 106.9)
- added HAT-Hole: VAL**, HAT-Hole, F.Cu at (107.5, 118.5)
- added HAT-Hole: VAL**, HAT-Hole, F.Cu at (107.5, 70.0)
- added HAT-Hole: VAL**, HAT-Hole, F.Cu at (165.5, 70.0)
- added HAT-Hole: VAL**, HAT-Hole, F.Cu at (165.5, 118.5)
- added IC1: ATMEGA1284P-P, DIP-40__600, F.Cu at (132.1, 95.2)
- added IC2: FT232RL, SSOP28, F.Cu at (160.0, 109.9)
- added IC3: CAT24C32, DIP-8__300, F.Cu at (163.3, 80.0)
- added J1: USB-B, HAR-M701-330442, F.Cu at (147.3, 118.7)
- added P1: CONN_20X2_STACKING, PIN_ARRAY_20X2, F.Cu at (136.5, 70.0)
- added P2: CONN_3, PIN_ARRAY_3X1, F.Cu at (152.4, 83.6)
- added P3: CONN_3, PIN_ARRAY_3X1, F.Cu at (110.5, 78.2)
- added P4: CONN_10X2, PIN_ARRAY_10x2, F.Cu at (116.8, 111.8)
- added P5: CONN_5, PIN_ARRAY_5x1, F.Cu at (119.9, 75.4)
- added P6: CONN_4, PIN_ARRAY_4x1, F.Cu at (144.5, 110.0)
- added R1: 10K, R3, F.Cu at (118.6, 116.6)
- added RES1: 20MHz, SIL-3, F.Cu at (161.0, 95.0)
- added SW1: SW_PUSH, TE1825910-6, F.Cu at (134.6, 111.8)
- added U1: SN74LVC1T45, SOT23_6, F.Cu at (134.6, 76.2)
- added U2: SN74LVC1T45, SOT23_6, F.Cu at (138.4, 76.2)
- added U3: SN74LVC1T45, SOT23_6, F.Cu at (142.2, 76.2)
Routing:
- net GND: track 0.00 -> 274.2 mm, vias 0 -> 1
- net Vcc: track 0.00 -> 194.7 mm, vias 0 -> 4
- net N-0000074: track 0.00 -> 61.7 mm, vias 0 -> 1
- net Vdd: track 0.00 -> 52.5 mm
- net MOSI50: track 0.00 -> 41.2 mm
- net RXD: track 0.00 -> 39.2 mm
- net MISO50: track 0.00 -> 39.1 mm
- net AP4: track 0.00 -> 38.4 mm
- net SCK50: track 0.00 -> 37.1 mm
- net AP3: track 0.00 -> 36.9 mm
- net AP2: track 0.00 -> 35.4 mm
- net AP1: track 0.00 -> 33.9 mm
- net DTR: track 0.00 -> 33.1 mm
- net TXD: track 0.00 -> 32.7 mm
- net IDSC: track 0.00 -> 30.3 mm
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- added copper zone on B.Cu, net (none)
- added copper zone on F.Cu, net (none)
Other:
- board text added: "10K"
- board text added: "4D Sys"
- board text added: "C1"
- board text added: "C2"
- board text added: "C3"
- board text added: "C4"
- board text added: "I2C"
- board text added: "IC1 ATMEGA1284P-P"
- board text added: "IC2 FT232RL"
- board text added: "IC3 CAT24C32"
- board text added: "J1"
- board text added: "P1"
- board text added: "P2"
- board text added: "P3"
- board text added: "P4"
- board text added: "P5"
- board text added: "P6"
- board text added: "RES1"
- board text added: "RPi I2C"
- board text added: "Rancho Hyrdoponics HydroHAT R1"
- board text added: "SN74LVC1T45 x3"
- board text added: "SW1"
- board text added: "U1"
- board text added: "U2"
- board text added: "U3"
