File: PTH PCB/HydroHAT.sch (KiCad schematic (older format))
At the start: 20 parts, among them IC1 ATMEGA1284P-P, IC2 FT232RL, IC3 CAT24C32, J1 USB-B, P1 CONN_20X2_STACKING, P2 CONN_3, P3 CONN_3, P4 CONN_10X2, P6 CONN_4, P7 CONN_5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

Commit message: PTH PCB Complete
Schematic also somewhat reworked.
Parts:
- renumbered P7 to P5
Connections:
- net GND: now also J1.5 (Shield_1), J1.6 (Shield_2)
- net AP1: now reaches P4.18 (P18)
- net AP1: now also IC1.26 ((PCINT20/TDO)PC4); no longer IC1.1 ((PCINT8/T0/XCK)PB0)
- net AP2: now reaches P4.16 (P16)
- net AP2: now also IC1.27 ((PCINT21/TDI)PC5); no longer IC1.2 ((PCINT9/CLKO/T1)PB1)
- net AP5: now reaches P4.10 (P10)
- net AP5: now also IC1.4 ((PCINT11/AIN1/OC0)PB3); no longer IC1.26 ((PCINT20/TDO)PC4)
- net AP6: now reaches P4.8 (P8)
- net AP6: now also IC1.3 ((PCINT10/AIN0/INT2)PB2); no longer IC1.27 ((PCINT21/TDI)PC5)
- net AP3: now reaches IC1.28 ((PCINT22/TOSC1)PC6)
- net AP3: now also P4.14 (P14); no longer P4.6 (P6)
- net AP4: now reaches IC1.29 ((PCINT23/TOSC2)PC7)
- net AP4: now also P4.12 (P12); no longer P4.4 (P4)
- new net AP7: IC1.2 ((PCINT9/CLKO/T1)PB1), P4.6 (P6)
- new net AP8: IC1.1 ((PCINT8/T0/XCK)PB0), P4.4 (P4)
- no-connect marks 54 -> 52
Changed lines of the file:
@@
 Sheet 1 1
 Title "HydroHAT Hydroponics Control Board"
-Date "25 sep 2014"
+Date "26 sep 2014"
 Rev "1"
 Comp "Rancho High School"
@@
 	4350 3300 4200 3300
 Wire Wire Line
-	6350 3400 7450 3400
-Wire Wire Line
-	7450 3400 7450 3200
-Wire Wire Line
-	7450 3200 7250 3200
-Wire Wire Line
-	6350 3500 7500 3500
-Wire Wire Line
-	7500 3500 7500 3100
-Wire Wire Line
-	7500 3100 7250 3100
-Wire Wire Line
-	6350 3600 7550 3600
-Wire Wire Line
-	7550 3600 7550 3000
-Wire Wire Line
-	7550 3000 7250 3000
-Wire Wire Line
-	6350 3700 7600 3700
-Wire Wire Line
-	7600 3700 7600 2900
-Wire Wire Line
-	7600 2900 7250 2900
-Wire Wire Line
-	6350 4700 7650 4700
-Wire Wire Line
-	7650 4700 7650 2800
-Wire Wire Line
-	7650 2800 7250 2800
-Wire Wire Line
-	6350 4800 7700 4800
-Wire Wire Line
-	7700 4800 7700 2700
-Wire Wire Line
-	7700 2700 7250 2700
-Wire Wire Line
-	6350 4900 7750 4900
-Wire Wire Line
-	7750 4900 7750 2600
-Wire Wire Line
-	7750 2600 7250 2600
-Wire Wire Line
-	6350 5000 7800 5000
-Wire Wire Line
-	7800 5000 7800 2500
-Wire Wire Line
-	7800 2500 7250 2500
-Wire Wire Line
 	6350 5400 6900 5400
 Wire Wire Line
@@
 	750  4300 850  4300
 NoConn ~ 850  4450
-NoConn ~ 850  4200
-NoConn ~ 1600 4200
 Text GLabel 1600 3850 1    60   Input ~ 0
 Vcc
@@
 IDSD
 $Comp
-L CONN_5 P7
+L CONN_5 P5
 U 1 1 542311A8
 P 9000 3100
-F 0 "P7" V 8950 3100 50  0000 C CNN
+F 0 "P5" V 8950 3100 50  0000 C CNN
 F 1 "CONN_5" V 9050 3100 50  0000 C CNN
 F 2 "" H 9000 3100 60  0000 C CNN
@@
 NoConn ~ 9900 5000
 NoConn ~ 9900 5200
+Wire Wire Line
+	850  4300 850  4150
+Wire Wire Line
+	850  4150 1600 4150
+Wire Wire Line
+	1600 4150 1600 4200
+Connection ~ 850  4200
+Text GLabel 6350 4700 2    60   Input ~ 0
+AP1
+Text GLabel 7250 3200 2    60   Input ~ 0
+AP1
+Text GLabel 7250 3100 2    60   Input ~ 0
+AP2
+Text GLabel 6350 4800 2    60   Input ~ 0
+AP2
+Text GLabel 6350 4900 2    60   Input ~ 0
+AP3
+Text GLabel 6350 5000 2    60   Input ~ 0
+AP4
+Text GLabel 7250 3000 2    60   Input ~ 0
+AP3
+Text GLabel 7250 2900 2    60   Input ~ 0
+AP4
+Text GLabel 7250 2800 2    60   Input ~ 0
+AP5
+Text GLabel 7250 2700 2    60   Input ~ 0
+AP6
+Text GLabel 7250 2600 2    60   Input ~ 0
+AP7
+Text GLabel 7250 2500 2    60   Input ~ 0
+AP8
+Text GLabel 6350 3700 2    60   Input ~ 0
+AP5
+Text GLabel 6350 3600 2    60   Input ~ 0
+AP6
+Text GLabel 6350 3500 2    60   Input ~ 0
+AP7
+Text GLabel 6350 3400 2    60   Input ~ 0
+AP8
 $EndSCHEMATC

Commit message: Added BOM And rejiggled some stuff
Parts:
- RES1: Distrib Link 490-1215-ND -> http://www.digikey.com/short/7tzm70
Changed lines of the file:
@@
 F 5 "CSTLS20M0X53-B0" H 4000 3100 60  0001 C CNN "MFG Part Num"
 F 6 "490-1215-ND" H 4000 3100 60  0001 C CNN "Distrib PN"
-F 7 "490-1215-ND" H 4000 3100 60  0001 C CNN "Distrib Link"
+F 7 "http://www.digikey.com/short/7tzm70" H 4000 3100 60  0001 C CNN "Distrib Link"
 	1    4000 3100
 	1    0    0    -1
